File: board/Rev0/pico2-nx-module/power.kicad_sch (KiCad schematic)
At the start: 10 parts, among them U5 AP61102QZ6-7

Commit message: layout update
Parts:
- L3: footprint (none) -> pico:DFE201610E
- TP3: footprint (none) -> TestPoint:TestPoint_Pad_1.0x1.0mm
Changed lines of the file:
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@@
 			)
 		)
-		(property "Footprint" ""
+		(property "Footprint" "TestPoint:TestPoint_Pad_1.0x1.0mm"
 			(at 180.34 95.25 0)
 			(effects
@@
 			)
 		)
-		(property "Footprint" ""
+		(property "Footprint" "pico:DFE201610E"
 			(at 160.02 95.25 0)
 			(effects
